Commit message: Actualizado hasta 29-05-2023

File: src/mmdt_rat20/urdf/esferitaNoInertiaPeque.xacro (robot description, xacro)
@@ -23,5 +23,5 @@
     <child link="esferaX_link"/>
     <axis xyz="1 0 0" />
-    <limit effort="1000.0" lower="-2" upper="10" velocity="0.5"/>
+    <limit effort="1000.0" lower="-100" upper="100" velocity="0.5"/>
     <origin rpy="0 0 0" xyz="0 0 0"/>
     <dynamics damping="1.0" friction="0.0"/>
@@ -31,5 +31,5 @@
     <child link="esferaY_link"/>
     <axis xyz="0 1 0" />
-    <limit effort="1000.0" lower="-2" upper="10" velocity="0.5"/>
+    <limit effort="1000.0" lower="-100" upper="100" velocity="0.5"/>
     <origin rpy="0 0 0" xyz="0 0 0"/>
     <dynamics damping="1.0" friction="0.0"/>
@@ -39,9 +39,9 @@
     <child link="esferaZ_link"/>
     <axis xyz="0 0 1" />
-    <limit effort="1000.0" lower="-2" upper="10" velocity="0.5"/>
+    <limit effort="1000.0" lower="-100" upper="100" velocity="0.5"/>
     <origin rpy="0 0 0" xyz="0 0 0"/>
     <dynamics damping="1.0" friction="0.0"/>
   </joint>
-<!-- AQUI SE DEFINE LAS CARACTERISTICAS FISICAS DE LA ESFERITA-->>
+<!-- AQUI SE DEFINE LAS CARACTERISTICAS FISICAS DE LA ESFERITA-->
   <link name="esferaX_link">
     <gravity>0</gravity>

File: src/mmdt_rat20/urdf/mmdt_rat20.urdf (robot description, URDF)
Before this commit: robot mmdt_rat20, 22 links, 21 joints
Joints:
- joint bEjeBaseTorso: limit lower=${-pi*0.5} upper=${pi*0.5} effort=1000 velocity=6.5 -> lower=-0.3 upper=0.3 effort=1000 velocity=6.5
- joint bEjeTorso: limit lower=${-pi} upper=${pi} effort=1000 velocity=6.5 -> lower=-0.3 upper=0.3 effort=1000 velocity=6.5
- joint camera_joint: origin xyz=0.2 -0.5 0.0 rpy=1.57 3.14 -0.4 -> xyz=0.15 -0.65 0.0 rpy=1.57 3.14 -0.4
