Commit message: Con Cambios para MMDT y control de dos brazos

File: src/mmdt_rat20/urdf/mesaDer.xacro (robot description, xacro)
@@ -39,5 +39,5 @@
     <!-- <collision name='collision'>
       <geometry>
-        <cylinder radius="1.5" length="0.02"/>
+        <cylinder radius="1.5" length="0.01"/>
       </geometry>
       <max_contacts>10</max_contacts>
@@ -58,5 +58,5 @@
       <origin xyz="0 0 0" rpy="0 0 0 "/>
       <geometry>
-        <cylinder radius="1.5" length="0.05"/>
+        <cylinder radius="1.5" length="0.01"/>
       </geometry>
       <origin xyz="0 0 0" rpy="0 0 0 "/>
@@ -102,5 +102,5 @@
     <mu1>0.2</mu1>
     <mu2>0.2</mu2>
-    <material>Gazebo/DarkGrey</material>
+    <material>Gazebo/Gold</material>
     <!-- <material>Table/Marble_Lightmap</material> -->
     <!-- <material>mmdt/pisoHierba</material>       -->

File: src/mmdt_rat20/urdf/mesaIzq.xacro (robot description, xacro)
@@ -4,4 +4,5 @@
   <xacro:property name="width" value="0.02" />
   <xacro:property name="radio" value="0.02" />
+  <xacro:property name="mass" value="1.0" />
   <!-- <xacro:include filename="$(find mmdt_rat20)/urdf/materials.xacro" /> -->
 <!-- DEFINICIONES INICIALES -->
@@ -37,7 +38,8 @@
       <pose>0 0 0 0 -0 0</pose>
     </inertial> -->
-    <collision name='collisionM'>
+    <!-- <collision name='collisionMI'> -->
+    <!-- <collision>
       <geometry>
-        <cylinder radius="1.5" length="0.05"/>
+        <cylinder radius="1.5" length="0.01"/>
       </geometry>
       <max_contacts>10</max_contacts>
@@ -45,5 +47,5 @@
         <contact>
           <ode/>
-        </contact>s
+        </contact>
         <bounce/>
         <friction>
@@ -54,9 +56,10 @@
         </friction>
       </surface>
-    </collision>
+    </collision> -->
+    <!-- <visual name='visual'> -->
     <visual>
       <origin xyz="0 0 0" rpy="0 0 0 "/>
       <geometry>
-        <cylinder radius="1.5" length="0.05"/>
+        <cylinder radius="1.5" length="0.01"/>
       </geometry>
       <origin xyz="0 0 0" rpy="0 0 0 "/>
@@ -72,4 +75,5 @@
     <kinematic>0</kinematic>
     <xacro:default_inertial mass="0.01"/>
+    <!-- <static>1</static> -->
   </link>
   <transmission name="gripper_extension_transZ" type="SimpleTransmission">
@@ -80,12 +84,32 @@
     <joint name="cilindroZ_extension">
       <hardwareInterface>EffortJointInterface</hardwareInterface>
+      <mechanicalReduction>1</mechanicalReduction>
     </joint>
   </transmission>
+    <!-- <transmission name="tran6_manipIzq">
+    <type>transmission_interface/SimpleTransmission</type>
+    <joint name="manipIzq_joint6">
+      <hardwareInterface>EffortJointInterface</hardwareInterface>
+    </joint>
+    <actuator name="motor6_manipIzq">
+      <hardwareInterface>EffortJointInterface</hardwareInterface>
+      <mechanicalReduction>1</mechanicalReduction>
+    </actuator>
+  </transmission> -->
   <!-- Gazebo plugin for ROS Control -->
   <gazebo>
+    <!-- <plugin name="gazebo_ros_control" filename="libgazebo_ros_control.so">
+    </plugin> -->
     <plugin name="gazebo_ros_control" filename="libgazebo_ros_control.so">
-      <!-- <robotNamespace>/cilindro</robotNamespace>
-      <robotSimType>gazebo_ros_control/DefaultRobotHWSim</robotSimType> -->
+      <!-- <robotNamespace>/cilindro</robotNamespace> -->
+      <robotSimType>gazebo_ros_control/DefaultRobotHWSim</robotSimType>
     </plugin>
+    <!-- <sensor name='my_contact' type='contact'>
+      <plugin name="my_plugin" filename="libcontact.so"/>
+      <contact>
+        <collision>collisionMI</collision>
+      </contact>
+      <update_rate>20</update_rate>
+    </sensor>-->
   </gazebo>
 <!-- **** Informacion de texturas:
@@ -102,14 +126,18 @@
     <mu1>0.2</mu1>
     <mu2>0.2</mu2>
-    <material>Gazebo/DarkGrey</material>
+    <material>Gazebo/Gold</material>
+    <!-- <material value="Gazebo/BlueTransparent"/> -->
     <!-- <material>Table/Marble_Lightmap</material> -->
     <!-- <material>mmdt/pisoHierba</material>       -->
-    <sensor name='my_contact' type='contact'>
-      <plugin name="my_plugin" filename="libcontact.so"/>
+    <!-- <plugin name="gazebo_ros_control" filename="libgazebo_ros_control.so">
+    </plugin> -->
+    <!-- <sensor name='my_contactI' type='contact'>
+      <always_on>true</always_on>
+      <plugin name="my_pluginI" filename="libcontact.so"/>
       <contact>
-        <collision>collisionM</collision>
+        <collision>collisionMI</collision>
       </contact>
-      <update_rate> 20 </update_rate>
-    </sensor>
+      <update_rate>20</update_rate>
+    </sensor> -->
   </gazebo>
 </robot>

File: src/mmdt_rat20/urdf/mmdt_rat20_CamarasDepth.urdf (robot description, URDF)
Before this commit: robot mmdt_rat20, 23 links, 22 joints
Joints:
- joint bEjeBaseTorso: limit lower=-1.57 upper=1.57 effort=1000 velocity=6.5 -> lower=-0.8 upper=0.8 effort=1000 velocity=6.5
- joint bEjeTorso: limit lower=0.0 upper=0.3 effort=1000 velocity=6.5 -> lower=0.0 upper=0.8 effort=1000 velocity=6.5
- joint manipDer_joint1: limit lower=-1.570796327 upper=1.570796327 effort=1000 velocity=6.5 -> lower=-3.14 upper=3.14 effort=1000 velocity=6.5
- joint manipDer_joint3: limit lower=-1.570796327 upper=1.570796327 effort=1000 velocity=6.5 -> lower=-1.570796327 upper=2.35 effort=1000 velocity=6.5
- joint manipDer_joint4: limit lower=-1.570796327 upper=1.570796327 effort=1000 velocity=6.5 -> lower=-3.14 upper=3.14 effort=1000 velocity=6.5
- joint manipIzq_joint1: limit lower=-1.570796327 upper=1.570796327 effort=1000 velocity=6.5 -> lower=-3.14 upper=3.14 effort=1000 velocity=6.5
- joint manipIzq_joint3: limit lower=-1.570796327 upper=1.570796327 effort=1000 velocity=6.5 -> lower=-1.570796327 upper=2.35 effort=1000 velocity=6.5
- joint manipIzq_joint4: limit lower=-1.570796327 upper=1.570796327 effort=1000 velocity=6.5 -> lower=-3.14 upper=3.14 effort=1000 velocity=6.5
